Commit message: Fix A1 bimanual joint limits

File: onerobotics_a1/urdf/a1_bimanual_stand.urdf (robot description, URDF)
Before this commit: robot onerobotics_a1_bimanual_stand, 17 links, 16 joints
Joints:
- joint joint_l1: limit lower=-3.14 upper=1.04 effort=0 velocity=0 -> lower=-3.14 upper=1.04 effort=15 velocity=30
- joint joint_l2: limit lower=-0.26 upper=3.14 effort=0 velocity=0 -> lower=-0.26 upper=3.14 effort=15 velocity=30
- joint joint_l3: limit lower=-2.75 upper=2.75 effort=0 velocity=0 -> lower=-2.75 upper=2.75 effort=15 velocity=30
- joint joint_l4: limit lower=-1.91 upper=1.91 effort=0 velocity=0 -> lower=-1.91 upper=1.91 effort=3 velocity=30
- joint joint_l5: limit lower=-2.75 upper=2.75 effort=0 velocity=0 -> lower=-2.75 upper=2.75 effort=3 velocity=30
- joint joint_l6: limit lower=-1.57 upper=1.57 effort=0 velocity=0 -> lower=-1.57 upper=1.57 effort=3 velocity=30
- joint joint_l7: limit lower=-2.75 upper=2.75 effort=0 velocity=0 -> lower=-2.75 upper=2.75 effort=3 velocity=30
- joint joint_r1: limit lower=-1.04 upper=3.14 effort=0 velocity=0 -> lower=-1.04 upper=3.14 effort=15 velocity=30
- joint joint_r2: limit lower=-3.14 upper=0.26 effort=0 velocity=0 -> lower=-3.14 upper=0.26 effort=15 velocity=30
- joint joint_r3: limit lower=-2.75 upper=2.75 effort=0 velocity=0 -> lower=-2.75 upper=2.75 effort=15 velocity=30
- joint joint_r4: limit lower=-1.91 upper=1.91 effort=0 velocity=0 -> lower=-1.91 upper=1.91 effort=3 velocity=30
- joint joint_r5: limit lower=-2.75 upper=2.75 effort=0 velocity=0 -> lower=-2.75 upper=2.75 effort=3 velocity=30
- joint joint_r6: limit lower=-1.57 upper=1.57 effort=0 velocity=0 -> lower=-1.57 upper=1.57 effort=3 velocity=30
- joint joint_r7: limit lower=-2.75 upper=2.75 effort=0 velocity=0 -> lower=-2.75 upper=2.75 effort=3 velocity=30

Commit message: Fix A1 bimanual terminal-link inertials

File: onerobotics_a1/urdf/a1_bimanual_stand.urdf (robot description, URDF)
Before this commit: robot onerobotics_a1_bimanual_stand, 17 links, 16 joints
Links:
- link Link_l7: mass 0.0177506448635751 -> 0.20
- link Link_r7: mass 0.0177506448635755 -> 0.20
